File: RTC/RTC.kicad_sch (KiCad schematic)
At the start: 13 parts, among them J1 Rasberry_to_stm, J2 Encoder R, J3 motor R, J4 Encoder L, J5 motor L, J6 Servo1, J7 Servo2, J8 Servo3, J9 Servo4, U2 L298N

Commit message: work all without Servo5 (rotation man)
Parts:
- added J10: Servo1, Connector_PinSocket_2.54mm:PinSocket_1x03_P2.54mm_Vertical, symbol Connector:Conn_01x03_Pin
- added J11: Power 12V, Connector_PinSocket_2.54mm:PinSocket_1x02_P2.54mm_Vertical, symbol Connector:Conn_01x02_Pin
- added U5: ~, User_Library:UBEC_POWER, symbol USERS:LM2896
- J1, J2, J4, U3, U4: footprint (none) -> Connector_PinSocket_2.54mm:PinSocket_1x04_P2.54mm_Vertical
- J3, J5: footprint (none) -> Connector_JST:JST_VH_B2P3-VH_1x02_P7.92mm_Vertical
- J6, J7, J8, J9: footprint (none) -> Connector_PinSocket_2.54mm:PinSocket_1x03_P2.54mm_Vertical
- U1: footprint (none) -> BlackPill:YAAJ_BlackPill_2
- U2: footprint Package_TO_SOT_THT:TO-220-15_P2.54x2.54mm_StaggerOdd_Lead4.58mm_Vertical -> User_Library:L298_Module
Connections:
- net 12v: now also J11.1 (Pin_1), U5. (Out-)
- net 5v: now also U1. (VB), J10.2 (Pin_2), U5. (Out-)
- net GND: now also U1. (VB), J10.1 (Pin_1), J11.2 (Pin_2), U5. (Out-)
- new net P_S_5: J10.3 (Pin_3), U1. (VB)
- no-connect marks 2 -> 19

Commit message: Work with PID on velocity
Parts:
- J1: value Rasberry_to_stm -> Raspberry_to_stm
- U3: value ~ -> Ultrasonic sensors
Other:
- added sheet LED (LED.kicad_sch)
- moved on the sheet: J1, J10, J11, J2, J3, J4, J5, J6, J7, J8, J9, U2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
